Commit message: added some materials. added 'odom' frame so base link can have an inertia

File: urdf/mallard_origins.urdf (robot description, URDF)
Before this commit: robot mallard_origins, 2 links, 1 joints
Links:
- added link odom
Joints:
- added joint odom_to_base_link: type fixed, parent odom, child base_link, origin xyz=0.15 0.0 0.0 rpy=0.0 0.0 0.0
