Commit message: spawning model in gazebo

File: urdf/01-chassis.urdf (robot description, URDF)
Before this commit: robot mallard_origins, 3 links, 2 joints
Links:
- removed link odom
- added link actuator, mass 2; collision cylinder length=0.1 radius=0.1; visual cylinder length=0.1 radius=0.1
Joints:
- removed joint odom_to_base_link
- added joint actuator_to_base_link: type continuous, parent base_link, child actuator, origin xyz=0.225 0.255 0.076 rpy=0 0 0, axis 0 1 0

Commit message: finished Mallard without thrusters. Attached two wheels as an example how to use them with Gazebo transmission and <gazebo> tag

File: urdf/01-chassis.urdf (robot description, URDF)
Before this commit: robot 02-actuators, 3 links, 2 joints
Joints:
- joint actuator_to_base_link: limit effort=30 velocity=1.0 -> (none)

File: urdf/03-actuator-velocity.urdf (robot description, URDF)
Before this commit: robot 02-actuators, 3 links, 2 joints
Links:
- removed link actuator
- added link wheel_1, mass 2; collision cylinder length=0.1 radius=0.2; visual cylinder length=0.1 radius=0.2
- added link wheel_2, mass 2; collision cylinder length=0.1 radius=0.2; visual cylinder length=0.1 radius=0.2
Joints:
- removed joint actuator_to_base_link
- added joint wheel_1_to_base_link: type continuous, parent base_link, child wheel_1, origin xyz=0.225 0.255 0.076 rpy=0 0 0, axis 0 1 0, limit effort=30 velocity=1.0
- added joint wheel_2_to_base_link: type continuous, parent base_link, child wheel_2, origin xyz=0.225 -0.255 0.076 rpy=0 0 0, axis 0 1 0, limit effort=30 velocity=1.0
