Commit message: initial commit on this branch

File: urdf/03-actuator-velocity.urdf (robot description, URDF)
Before this commit: robot mallard, 4 links, 3 joints
Links:
- removed link wheel_1
- removed link wheel_2
Joints:
- removed joint wheel_1_to_base_link
- removed joint wheel_2_to_base_link

File: urdf/mallard_thrusters.xacro (robot description, xacro)
@@ -1,4 +1,4 @@
 <?xml version="1.0"?>
-<robot name="mallard_origins">
+<robot name="mallard">
   <material name="blue">
     <color rgba="0.0 0.0 0.8 1.0"/>
@@ -13,9 +13,4 @@
     <color rgba="0.8 0.8 0.8 1.0"/>
   </material>
-  <!-- <link name="odom">
-    <geometry>
-      <box size="0.001 0.001 0.001"/>
-    </geometry>
-  </link> -->
   <link name="base_link">
       <!-- Channels (aluminum connecting elements) -->
@@ -76,9 +71,4 @@
       </inertial>
   </link>
-  <!-- <joint name="odom_to_base_link" type="fixed">
-    <origin xyz="0.15 0.0 0.0" rpy="0.0 0.0 0.0"/>
-    <parent link="odom"/>
-    <child link="base_link"/>
-  </joint> -->
   <link name="lidar">
     <visual name="lidar_base">
@@ -118,29 +108,3 @@
     <origin xyz="0.225 0.0 0.152" rpy="0.0 0.0 0.0"/>
   </joint>
-  <link name="actuator">
-     <!-- need physics (colision, inertia) for gazebo to work !!!! -->
-      <visual name="actuator_visual">
-          <geometry>
-              <cylinder radius="0.1" length="0.1"/>
-          </geometry>
-          <material name="black"/>
-          <origin xyz="0.0 0.05 0.0" rpy="1.5707 0.0 0.0"/>
-      </visual>
-      <collision name="actuator_collision">
-          <geometry>
-              <cylinder radius="0.1" length="0.1"/>
-          </geometry>
-          <origin xyz="0.0 0.05 0.0" rpy="1.5707 0.0 0.0"/>
-      </collision>
-      <inertial>
-        <mass value="2"/>
-        <inertia ixx="1.0" ixy="0.0" ixz="0.0" iyy="1.0" iyz="0.0" izz="1.0"/>
-    </inertial>
-  </link>
-  <joint name="actuator_to_base_link" type="continuous">
-      <parent link="base_link"/>
-      <child link="actuator"/>
-      <axis xyz="0 1 0" rpy="0 0 0"/>
-      <origin xyz="0.225 0.255 0.076" rpy="0 0 0"/>
-  </joint>
 </robot>
