Commit message: solved Mallards body inertia, and <compensation> tag calculations. Mallard behaves more realistically now

File: urdf/mallard_thrusters.xacro (robot description, xacro)
@@ -26,5 +26,5 @@
           <child link="${name}"/>
           <origin rpy="${rpy}" xyz="${xyz}"/>
-          <dynamics damping="10.0"/>
+          <dynamics damping="1.0"/>
           <axis xyz="0 1 0"/>
           <limit effort="30" velocity="5.0" lower="-${PI}" upper="${PI}" />
@@ -50,11 +50,11 @@
           </visual>
           <inertial>
-              <mass  value="0.5"/>
-              <inertia ixx="0.1"
+              <mass  value="0.3"/>
+              <inertia ixx="0.001"
                        ixy="0.0"
                        ixz="0.0"
-                       iyy="0.1"
+                       iyy="0.001"
                        iyz="0.0"
-                       izz="0.1"/>
+                       izz="0.001"/>
           </inertial>
       </link>
@@ -63,8 +63,5 @@
       </gazebo>
       <buoyancy>
-          <compensation>1.01</compensation>
-          <!-- <origin xyz= "0 0 0"/>
-          <limit radius="0.0"/>
-          <damping xyz="60 100 100" rpy="20 50 50"/> -->
+          <compensation>0.6</compensation>
       </buoyancy>
   </xacro:macro>
@@ -78,11 +75,12 @@
         </geometry>
         <material name="gray"/>
-        <origin rpy="0 0 0" xyz="0 -0.15 0"/>
+        <origin  xyz="0 -0.15 0" rpy="0 0 0"/>
       </visual>
-      <collision name="r_channel_collision">
+      <collision name="mallard_box">
+        <origin xyz="0 0 0.057" rpy="0 0 0"/>
         <geometry>
-          <box size="0.450 0.038 0.038"/>
+          <box size="0.564 0.5 0.152"/>
         </geometry>
-        <origin rpy="0 0 0" xyz="0 -0.15 0"/>
+        <!-- <origin rpy="0 0 0" xyz="0 0 0"/>  -->
       </collision>
       <visual name="l_channel_visual">
@@ -90,12 +88,6 @@
           <box size="0.450 0.038 0.038"/>
         </geometry>
-        <origin rpy="0 0 0" xyz="0 0.15 0"/>
+        <origin xyz="0 0.15 0" rpy="0 0 0"/>
       </visual>
-      <collision name="l_channel_collision">
-        <geometry>
-          <box size="0.450 0.038 0.038"/>
-        </geometry>
-        <origin rpy="0 0 0" xyz="0 0.15 0"/>
-      </collision>
       <!-- Cylinders (acrylic tubes)-->
       <visual name="front_tube_visual">
@@ -105,10 +97,4 @@
         <origin xyz="0.225 0 0.076" rpy="1.5707 0.0 0.0"/>
       </visual>
-      <collision name="front_tube_collision">
-        <geometry>
-          <cylinder radius="0.057" length="0.5"/>
-        </geometry>
-        <origin xyz="0.225 0 0.076" rpy="1.5707 0.0 0.0"/>
-      </collision>
       <visual name="rear_tube_visual">
         <geometry>
@@ -117,13 +103,8 @@
         <origin xyz="-0.225 0 0.076" rpy="1.5707 0.0 0.0"/>
       </visual>
-      <collision name="rear_tube_collision">
-        <geometry>
-          <cylinder radius="0.057" length="0.5"/>
-        </geometry>
-        <origin xyz="-0.225 0 0.076" rpy="1.5707 0.0 0.0"/>
-      </collision>
       <!-- chassis physics -->
       <inertial>
-        <mass value="10.0"/>
+        <origin xyz="0 0 -0.019" rpy="0 0 0"/>
+        <mass value="10.5"/>
         <inertia ixx="0.17" ixy="0.0" ixz="0.0" iyy="0.25" iyz="0.0" izz="0.40"/>
       </inertial>
@@ -131,8 +112,10 @@
       begins to decrease when approaching the water surface -->
       <buoyancy>
-          <compensation>1.00</compensation>
+          <!-- Compensation coefficient is buoyancy force to weight ratio. Mallard
+               buoyancy force is 11.52kg, weight is10.5kg.   -->
+          <compensation>1.1</compensation>
           <origin xyz= "0 0 0"/>
           <limit radius="0.0"/>
-          <damping xyz="60 100 100" rpy="20 50 50"/>
+          <damping xyz="80 100 100" rpy="20 50 50"/>
       </buoyancy>
   </link>
