Commit message: Moved lidar link to separate file. Sorted gazebo colors - the <visual> tags can not have names otherwise it doesnt work

File: urdf/ballast.xacro (robot description, xacro)
@@ -8,5 +8,5 @@
                     <cylinder radius="0.05" length="0.01"/>
                 </geometry>
-                <material name="red">
+                <material name="blue">
                     <color rgba="0.8 0.0 0.0 1.0"/>
                 </material>
@@ -22,4 +22,7 @@
             <child link="${name}"/>
         </joint>
+        <gazebo reference="${name}">
+          <material>Gazebo/Blue</material>
+      </gazebo>
     </xacro:macro>
 </robot>

File: urdf/mallard_main.xacro (robot description, xacro)
@@ -1,4 +1,5 @@
 <?xml version="1.0"?>
 <robot name="mallard" xmlns:xacro="http://www.ros.org/wiki/xacro">
+  <xacro:include filename="lidar.xacro"/>
   <xacro:include filename="ballast.xacro"/>
   <xacro:include filename="thruster.xacro"/>
@@ -21,52 +22,7 @@
     <color rgba="0.8 0.8 0.8 1.0"/>
   </material> -->
-  <!--  *** MACROS *** -->
-  <!-- Thruster link -->
-  <!-- <xacro:macro name="thruster_link" params="name xyz rpy">
-      <joint name="${name}" type="revolute">
-          <parent link="base_link"/>
-          <child link="${name}"/>
-          <origin xyz="${xyz}" rpy="${rpy}"/>
-          <dynamics damping="1.0"/>
-          <axis xyz="0 1 0"/>
-          <limit effort="30" velocity="5.0" lower="-${PI}" upper="${PI}" />
-      </joint>
-      <link name="${name}">
-          <visual name="${name}_1">
-              <geometry>
-                  <cylinder length="${tl1}" radius="${tr1}"/>
-              </geometry>
-              <material name="blue">
-                  <color rgba="0 0 0.8 1"/>
-              </material>
-          </visual>
-          <visual name="${name}_2">
-              <origin xyz="0 0 ${tl2/4}"/>
-              <geometry>
-                  <cylinder length="${tl2}" radius="${tr2}"/>
-              </geometry>
-              <material name="black">
-                <color rgba="0 0 0 1"/>
-              </material>
-          </visual>
-          <inertial>
-              <mass  value="0.3"/>
-              <inertia ixx="0.001"
-                       ixy="0.0"
-                       ixz="0.0"
-                       iyy="0.001"
-                       iyz="0.0"
-                       izz="0.001"/>
-          </inertial>
-      </link>
-      <gazebo reference="${name}">
-          <material>Gazebo/Black</material>
-      </gazebo>
-      <buoyancy>
-          <compensation>0.6</compensation>
-      </buoyancy>
-  </xacro:macro>  -->
-  <!-- <link name="odom">
-  </link> -->
+  <gazebo reference="base_link">
+      <material>Gazebo/Blue</material>
+  </gazebo>
   <link name="base_link">
       <!-- Channels (aluminum connecting elements) -->
@@ -85,5 +41,4 @@
           <box size="0.564 0.5 0.152"/>
         </geometry>
-        <!-- <origin rpy="0 0 0" xyz="0 0 0"/>  -->
       </collision>
       <visual name="l_channel_visual">
@@ -123,50 +78,5 @@
       </buoyancy>
   </link>
-  <!-- <joint name="odom_to_base_link" type="fixed">
-    <origin xyz="0.5 0.0 0.0" rpy="0.0 0.0 0.0"/>
-    <parent link="odom"/>
-    <child link="base_link"/>
-  </joint> -->
-  <link name="lidar">
-    <visual name="lidar_base">
-      <geometry>
-        <box size="0.06 0.061 0.048"/>
-      </geometry>
-      <material name="blue">
-        <color rgba="0.0 0.0 0.8 1.0"/>
-      </material>
-      <origin xyz="0.0 0.0 0.0"/>
-    </visual>
-    <collision>
-      <geometry>
-        <box size="0.06 0.061 0.048"/>
-      </geometry>
-      <origin xyz="0.0 0.0 0.0"/>
-    </collision>
-    <visual name="optical_hood">
-      <origin xyz="0 0 0.0425"/>
-      <geometry>
-        <cylinder radius="0.025" length="0.037"/>
-      </geometry>
-      <material name="blue">
-        <color rgba="0.0 0.0 0.8 1.0"/>
-      </material>
-    </visual>
-    <collision>
-      <origin xyz="0.0 0.0 0.048"/>
-      <geometry>
-        <cylinder radius="0.025" length="0.037"/>
-      </geometry>
-    </collision>
-    <inertial>
-      <mass value="0.3"/>
-      <inertia ixx="0.00020" ixy="0.0" ixz="0.0" iyy="0.00020" iyz="0.0" izz="0.00015"/>
-    </inertial>
-  </link>
-  <joint name="lidar_to_base_link" type="fixed">
-    <parent link="base_link"/>
-    <child link="lidar"/>
-    <origin xyz="0.225 0 0.152"/>
-  </joint>
+  <xacro:lidar name="sick_lidar" mass="0.27" xyz="0.225 0 0.152"/>
   <!-- Ballast -->
   <xacro:ballast name="ballast_1" mass="0.14" xyz=" 0.225 -0.25 0.076" rpy="${PI/2} 0 0"/>

File: urdf/thruster.xacro (robot description, xacro)
@@ -24,6 +24,6 @@
                   <cylinder length="${tl2}" radius="${tr2}"/>
               </geometry>
-              <material name="black">
-                <color rgba="0 0 0 1"/>
+              <material name="blue">
+                 <color rgba="0 0 0.8 1"/>
               </material>
           </visual>
@@ -39,5 +39,5 @@
       </link>
       <gazebo reference="${name}">
-          <material>Gazebo/Black</material>
+          <material>Gazebo/Blue</material>
       </gazebo>
       <buoyancy>
