Commit message: last commit before switch to new branch

File: urdf/lidar_sensor.xacro (robot description, xacro)
@@ -26,10 +26,10 @@
             <sensor type="ray" name="head_hokuyo_sensor">
                 <pose>0 0 0 0 0 0</pose>
-                <visualize>true</visualize>
+                <visualize>false</visualize>
                 <update_rate>${update_rate}</update_rate>
                 <ray>
                     <scan>
                         <horizontal>
-                            <samples>50</samples>
+                            <samples>100</samples>
                             <resolution>1.0</resolution>
                             <min_angle>${-3*PI/4}</min_angle>
@@ -38,7 +38,7 @@
                     </scan>
                   <range>
-                      <min>0.01</min>
-                      <max>10.0</max>
-                      <resolution>0.005</resolution>
+                      <min>0.05</min>
+                      <max>25.0</max>
+                      <resolution>0.33</resolution>
                   </range>
                   <noise>

File: urdf/mallard_main.xacro (robot description, xacro)
@@ -1,8 +1,9 @@
 <?xml version="1.0"?>
 <robot name="mallard" xmlns:xacro="http://www.ros.org/wiki/xacro">
-  <xacro:include filename="lidar_body.xacro"/>
-  <xacro:include filename="lidar_sensor.xacro"/>
-  <xacro:include filename="ballast.xacro"/>
-  <xacro:include filename="thruster.xacro"/>
+  <xacro:include filename="$(find mallard_urdf)/urdf/lidar_sensor.xacro"/>
+  <xacro:include filename="$(find mallard_urdf)/urdf/lidar_body.xacro"/>
+  <!-- <xacro:include filename="lidar_sensor.xacro"/> -->
+  <xacro:include filename="$(find mallard_urdf)/urdf/ballast.xacro"/>
+  <xacro:include filename="$(find mallard_urdf)/urdf/thruster.xacro"/>
   <!-- Thrusters components & constants -->
   <xacro:property name="PI" value="3.1415926535897931"/>
@@ -85,5 +86,5 @@
 		lidar_topic="mallard/lidar_data"
 		update_rate="100">
-		<origin xyz="0 0 0.068" rpy="0 0 0"/>
+		<origin xyz="0 0 0.044" rpy="0 0 0"/>
 	</xacro:LIDAR>
   <!-- Ballast -->

Commit message: removed lidar_body and put it in lidar.xacro. moved the scan of the laser from paren to child, i.e. lidar_name parameter in framename and bodyframe parameters

File: urdf/lidar_sensor.xacro (robot description, xacro)
@@ -2,5 +2,5 @@
 <robot xmlns:xacro="http://www.ros.org/wiki/xacro" name="mallard">
     <xacro:property name="PI" value="3.1415926535897931"/>
-    <xacro:macro name="LIDAR" params="parent lidar_name lidar_topic update_rate *origin">
+    <xacro:macro name="lidar" params="parent lidar_name mass lidar_topic update_rate *origin">
         <joint name="${lidar_name}_joint" type="fixed">
             <xacro:insert_block name="origin"/>
@@ -9,8 +9,4 @@
         </joint>
         <link name="${lidar_name}">
-            <inertial>
-                <mass value="0.010"/>
-                <inertia ixx="0" iyy="0" izz="0" ixy="0" ixz="0" iyz="0"/>
-            </inertial>
             <visual>
                 <geometry>
@@ -21,4 +17,17 @@
                 </material>
             </visual>
+            <visual>
+                <origin xyz="0 0 -0.044"/>
+                <geometry>
+                    <box size="0.06 0.061 0.048"/>
+                </geometry>
+                <material name="blue">
+                    <color rgba="0.0 0.0 0.8 1.0"/>
+                </material>
+            </visual>
+            <inertial>
+                <mass value="${mass}"/>
+                <inertia ixx="0.00020" ixy="0.0" ixz="0.0" iyy="0.00020" iyz="0.0" izz="0.00015"/>
+            </inertial>
         </link>
         <gazebo reference="${lidar_name}">
@@ -26,11 +35,11 @@
             <sensor type="ray" name="head_hokuyo_sensor">
                 <pose>0 0 0 0 0 0</pose>
-                <visualize>false</visualize>
+                <visualize>true</visualize>
                 <update_rate>${update_rate}</update_rate>
                 <ray>
                     <scan>
                         <horizontal>
-                            <samples>100</samples>
-                            <resolution>1.0</resolution>
+                            <samples>800</samples>
+                            <resolution>1</resolution>
                             <min_angle>${-3*PI/4}</min_angle>
                             <max_angle>${3*PI/4}</max_angle>
@@ -40,5 +49,5 @@
                       <min>0.05</min>
                       <max>25.0</max>
-                      <resolution>0.33</resolution>
+                      <resolution>0.01</resolution>
                   </range>
                   <noise>
@@ -53,6 +62,8 @@
                     <update_rate>${update_rate}</update_rate>
                     <topicName>${lidar_topic}</topicName>
-                    <frameName>${parent}</frameName>
-                    <bodyName>${parent}</bodyName>
+                    <!-- <frameName>${parent}</frameName>
+                    <bodyName>${parent}</bodyName> -->
+                    <frameName>${lidar_name}</frameName>
+                    <bodyName>${lidar_name}</bodyName>
                 </plugin>
             </sensor>

File: urdf/mallard_main.xacro (robot description, xacro)
@@ -2,5 +2,5 @@
 <robot name="mallard" xmlns:xacro="http://www.ros.org/wiki/xacro">
   <xacro:include filename="$(find mallard_urdf)/urdf/lidar_sensor.xacro"/>
-  <xacro:include filename="$(find mallard_urdf)/urdf/lidar_body.xacro"/>
+  <!-- <xacro:include filename="$(find mallard_urdf)/urdf/lidar_body.xacro"/> -->
   <!-- <xacro:include filename="lidar_sensor.xacro"/> -->
   <xacro:include filename="$(find mallard_urdf)/urdf/ballast.xacro"/>
@@ -12,19 +12,12 @@
   <xacro:property name="tr2" value=".047" />
   <xacro:property name="tl2" value=".045" />
-  <!-- <material name="blue">
-    <color rgba="0.0 0.0 0.8 1.0"/>
-  </material>
-  <material name="black">
-    <color rgba="0.0 0.0 0.0 1.0"/>
-  </material>
-  <material name="red">
-    <color rgba="0.8 0.0 0.0 1.0"/>
-  </material>
-  <material name="gray">
-    <color rgba="0.8 0.8 0.8 1.0"/>
-  </material> -->
   <gazebo reference="base_link">
       <material>Gazebo/Blue</material>
   </gazebo>
+  <!-- <link name="odom">
+    <geometry>
+      <box size="0.01 0.01 0.01"/>
+    </geometry>
+  </link> -->
   <link name="base_link">
       <!-- Channels (aluminum connecting elements) -->
@@ -80,12 +73,18 @@
       </buoyancy>
   </link>
-  <xacro:lidar_body name="lidar_body" mass="0.27" xyz="0.225 0 0.152"/>
-  <xacro:LIDAR
-		parent="lidar_body"
-		lidar_name="urg_lidar"
-		lidar_topic="mallard/lidar_data"
-		update_rate="100">
-		<origin xyz="0 0 0.044" rpy="0 0 0"/>
-	</xacro:LIDAR>
+  <!-- <joint name="odom_to_base_link" type="fixed">
+    <origin xyz="0.0 0.0 0.0" rpy="0.0 0.0 0.0"/>
+    <parent link="odom"/>
+    <child link="base_link"/>
+  </joint> -->
+  <!-- <xacro:lidar_body name="lidar_base" mass="0.27" xyz="0.225 0 0.152"/> -->
+  <xacro:lidar
+		parent="base_link"
+		lidar_name="laser"
+    mass="0.27"
+		lidar_topic="scan"
+		update_rate="15">
+		<origin xyz="0.225 0 0.194"/>
+	</xacro:lidar>
   <!-- Ballast -->
   <xacro:ballast name="ballast_1" mass="0.14" xyz=" 0.225 -0.25 0.076" rpy="${PI/2} 0 0"/>
