Commit message: Added pond, 4x3x1.4m  and removed the ship background. Added lidar from Wilson xacro. removed top hood from lidar's body.

File: urdf/control_thrusters.urdf (robot description, URDF)
Before this commit: robot thrusters, 0 links, 4 joints
Joints:
- joint x_thr_left: limit lower=-7 upper=10 -> lower=-2 upper=2
- joint x_thr_right: limit lower=-7 upper=10 -> lower=-2 upper=2
- joint y_thr_left: limit lower=-7 upper=10 -> lower=-2 upper=2
- joint y_thr_right: limit lower=-7 upper=10 -> lower=-2 upper=2

File: urdf/lidar_body.xacro (robot description, xacro)
@@ -1,5 +1,5 @@
 <?xml version="1.0"?>
 <robot xmlns:xacro="http://www.ros.org/wiki/xacro" name="mallard">
-    <xacro:macro name="lidar" params="name mass xyz">
+    <xacro:macro name="lidar_body" params="name mass xyz">
     <link name="${name}">
     <visual>
@@ -12,25 +12,4 @@
       <origin xyz="0.0 0.0 0.0"/>
     </visual>
-    <collision>
-      <geometry>
-        <box size="0.06 0.061 0.048"/>
-      </geometry>
-      <origin xyz="0.0 0.0 0.0"/>
-    </collision>
-    <visual>
-      <origin xyz="0 0 0.0425"/>
-      <geometry>
-        <cylinder radius="0.025" length="0.037"/>
-      </geometry>
-      <material name="blue">
-        <color rgba="0.0 0.0 0.8 1.0"/>
-      </material>
-    </visual>
-    <collision>
-      <origin xyz="0.0 0.0 0.048"/>
-      <geometry>
-        <cylinder radius="0.025" length="0.037"/>
-      </geometry>
-    </collision>
     <inertial>
       <mass value="${mass}"/>

File: urdf/mallard_main.xacro (robot description, xacro)
@@ -1,5 +1,6 @@
 <?xml version="1.0"?>
 <robot name="mallard" xmlns:xacro="http://www.ros.org/wiki/xacro">
-  <xacro:include filename="lidar.xacro"/>
+  <xacro:include filename="lidar_body.xacro"/>
+  <xacro:include filename="lidar_sensor.xacro"/>
   <xacro:include filename="ballast.xacro"/>
   <xacro:include filename="thruster.xacro"/>
@@ -75,8 +76,15 @@
           <origin xyz= "0 0 0"/>
           <limit radius="0.1"/>
-          <damping xyz="100 100 100" rpy="2 2 2"/>
+          <damping xyz="120 120 120" rpy="2 2 2"/>
       </buoyancy>
   </link>
-  <xacro:lidar name="sick_lidar" mass="0.27" xyz="0.225 0 0.152"/>
+  <xacro:lidar_body name="lidar_body" mass="0.27" xyz="0.225 0 0.152"/>
+  <xacro:LIDAR
+		parent="lidar_body"
+		lidar_name="urg_lidar"
+		lidar_topic="mallard/lidar_data"
+		update_rate="100">
+		<origin xyz="0 0 0.068" rpy="0 0 0"/>
+	</xacro:LIDAR>
   <!-- Ballast -->
   <xacro:ballast name="ballast_1" mass="0.14" xyz=" 0.225 -0.25 0.076" rpy="${PI/2} 0 0"/>
@@ -98,17 +106,17 @@
                         the thruster name is the name of the corresponding link -->
                 <thruster>
-                    <effort>10</effort>
+                    <effort>2</effort>
                     <name>x_thr_left</name>
                 </thruster>
                 <thruster>
-                    <effort>10</effort>
+                    <effort>2</effort>
                     <name>x_thr_right</name>
                 </thruster>
                 <thruster>
-                    <effort>10</effort>
+                    <effort>2</effort>
                     <name>y_thr_left</name>
                 </thruster>
                 <thruster>
-                    <effort>10</effort>
+                    <effort>2</effort>
                     <name>y_thr_right</name>
                 </thruster>
@@ -117,5 +125,5 @@
                 <thruster>
                     <map>0 1 0 0 0 0</map>
-                    <effort>10</effort>
+                    <effort>2</effort>
                 </thruster>
       </plugin>

Commit message: rotated 'y' thrusters by 180 degrees to correspond to real mallard. moved kgstripes, kglocal and kguseful to auxiliary folder. Had to add __init__.py inside that folder so python nows where the files are

File: urdf/control_thrusters.urdf (robot description, URDF)
Before this commit: robot thrusters, 0 links, 4 joints
Joints:
- joint x_thr_left: limit lower=-2 upper=2 -> lower=-7 upper=10
- joint x_thr_right: limit lower=-2 upper=2 -> lower=-7 upper=10
- joint y_thr_left: limit lower=-2 upper=2 -> lower=-7 upper=10
- joint y_thr_right: limit lower=-2 upper=2 -> lower=-7 upper=10

File: urdf/lidar_sensor.xacro (robot description, xacro)
@@ -35,5 +35,5 @@
             <sensor type="ray" name="head_hokuyo_sensor">
                 <pose>0 0 0 0 0 0</pose>
-                <visualize>true</visualize>
+                <visualize>false</visualize>
                 <update_rate>${update_rate}</update_rate>
                 <ray>

File: urdf/mallard_main.xacro (robot description, xacro)
@@ -81,6 +81,6 @@
   <xacro:thruster_link name="x_thr_right"  xyz="${(tl1/2)-0.188} -0.207 -0.041" rpy="0 ${-PI/2} 0"/>
   <!-- Side thrusters -->
-  <xacro:thruster_link name="y_thr_right"   xyz=" 0.233 ${0.114-(tl1/2)} -0.041" rpy="0 ${PI/2} ${-PI/2}"/>
-  <xacro:thruster_link name="y_thr_left"  xyz="-0.233 ${0.114-(tl1/2)} -0.041" rpy="0 ${PI/2} ${-PI/2}"/>
+  <xacro:thruster_link name="y_thr_right"   xyz=" 0.233 ${0.114-(tl1/2)} -0.041" rpy="0 ${PI/2} ${PI/2}"/>
+  <xacro:thruster_link name="y_thr_left"  xyz="-0.233 ${0.114-(tl1/2)} -0.041" rpy="0 ${PI/2} ${PI/2}"/>
   <!-- FreeFloating plugin -->
   <gazebo>
@@ -93,17 +93,17 @@
                         the thruster name is the name of the corresponding link -->
                 <thruster>
-                    <effort>2</effort>
+                    <effort>10</effort>
                     <name>x_thr_left</name>
                 </thruster>
                 <thruster>
-                    <effort>2</effort>
+                    <effort>10</effort>
                     <name>x_thr_right</name>
                 </thruster>
                 <thruster>
-                    <effort>2</effort>
+                    <effort>10</effort>
                     <name>y_thr_left</name>
                 </thruster>
                 <thruster>
-                    <effort>2</effort>
+                    <effort>10</effort>
                     <name>y_thr_right</name>
                 </thruster>
