Commit message: edited README file. Added basic Rviz launch for urdf editing.

File: urdf/mallard_main.xacro (robot description, xacro)
@@ -5,6 +5,6 @@
   <xacro:property name="tr1" value=".02" />
   <xacro:property name="tl1" value=".1" />
-  <xacro:property name="tr2" value=".05" />
-  <xacro:property name="tl2" value=".03" />
+  <xacro:property name="tr2" value=".047" />
+  <xacro:property name="tl2" value=".045" />
   <material name="blue">
     <color rgba="0.0 0.0 0.8 1.0"/>
@@ -117,5 +117,5 @@
           <origin xyz= "0 0 0"/>
           <limit radius="0.0"/>
-          <damping xyz="50 50 100" rpy="1 1 1"/>
+          <damping xyz="30 30 80" rpy="1 1 1"/>
       </buoyancy>
   </link>

Commit message: added two, side thrusters. They need to be fixed to work in gazebo as weel

File: urdf/mallard_main.xacro (robot description, xacro)
@@ -25,5 +25,5 @@
           <parent link="base_link"/>
           <child link="${name}"/>
-          <origin rpy="${rpy}" xyz="${xyz}"/>
+          <origin xyz="${xyz}" rpy="${rpy}"/>
           <dynamics damping="1.0"/>
           <axis xyz="0 1 0"/>
@@ -36,15 +36,16 @@
                   <cylinder length="${tl1}" radius="${tr1}"/>
               </geometry>
-              <material name="black">
-                  <color rgba="0 0 0 1"/>
+              <material name="blue">
+                  <color rgba="0 0 0.8 1"/>
               </material>
           </visual>
           <visual name="${name}_2">
-              <origin xyz="0 0 ${(tl1+tl2)/2}"/>
+              <!-- <origin xyz="0 0 ${(tl1+tl2)/2}"/> -->
+              <origin xyz="0 0 ${tl2/4}"/>
               <geometry>
                   <cylinder length="${tl2}" radius="${tr2}"/>
               </geometry>
               <material name="black">
-                  <color rgba="0 0 0 1"/>
+                <color rgba="0 0 0 1"/>
               </material>
           </visual>
@@ -117,5 +118,5 @@
           <origin xyz= "0 0 0"/>
           <limit radius="0.0"/>
-          <damping xyz="30 30 80" rpy="1 1 1"/>
+          <damping xyz="50 50 80" rpy="1 1 1"/>
       </buoyancy>
   </link>
@@ -162,7 +163,10 @@
     <origin xyz="0.225 0.0 0.152" rpy="0.0 0.0 0.0"/>
   </joint> -->
-  <!-- Make four thrusters -->
-  <xacro:thruster_link name="x_thr_left"   xyz="0  0.2 -0.05" rpy="0 ${-PI/2} 0"/>
-  <xacro:thruster_link name="x_thr_right"  xyz="0  -0.2 -0.05" rpy="0 ${-PI/2} 0"/>
+  <!-- Forward thrusters -->
+  <xacro:thruster_link name="x_thr_left"   xyz="${(tl1/2)-0.188}  0.207 -0.041" rpy="0 ${-PI/2} 0"/>
+  <xacro:thruster_link name="x_thr_right"  xyz="${(tl1/2)-0.188} -0.207 -0.041" rpy="0 ${-PI/2} 0"/>
+  <!-- Side thrusters -->
+  <xacro:thruster_link name="y_thr_left"   xyz=" 0.233 ${0.114-(tl1/2)} -0.041" rpy="0 ${PI/2} ${-PI/2}"/>
+  <xacro:thruster_link name="y_thr_right"  xyz="-0.233 ${0.114-(tl1/2)} -0.041" rpy="0 ${PI/2} ${-PI/2}"/>
   <!-- FreeFloating plugin -->
   <gazebo>

Commit message: added and checked in gazebo and rviz two side thrusters. Orientation and positioning is as close to real Mallard as possible, which translates to physics because the tube where lidar suppose to be is lifted, due to weight of three trhusters on the other tube. It looks very realistic.

File: urdf/mallard_main.xacro (robot description, xacro)
@@ -115,5 +115,5 @@
           <!-- Compensation coefficient is buoyancy force to weight ratio. Mallard
                buoyancy force is 11.52kg, weight is10.5kg.   -->
-          <compensation>1.1</compensation>
+          <compensation>1.2</compensation>
           <origin xyz= "0 0 0"/>
           <limit radius="0.0"/>
@@ -179,10 +179,18 @@
                         the thruster name is the name of the corresponding link -->
                 <thruster>
-                    <effort>30</effort>
+                    <effort>10</effort>
                     <name>x_thr_left</name>
                 </thruster>
                 <thruster>
-                    <effort>30</effort>
+                    <effort>10</effort>
                     <name>x_thr_right</name>
+                </thruster>
+                <thruster>
+                    <effort>10</effort>
+                    <name>y_thr_left</name>
+                </thruster>
+                <thruster>
+                    <effort>10</effort>
+                    <name>y_thr_right</name>
                 </thruster>
                 <!-- <map> describes where the force or torque is applied
@@ -190,5 +198,5 @@
                 <thruster>
                     <map>0 1 0 0 0 0</map>
-                    <effort>30</effort>
+                    <effort>10</effort>
                 </thruster>
       </plugin>

File: urdf/mallard_thrusters.urdf (robot description, URDF)
Before this commit: robot thrusters, 0 links, 2 joints
Joints:
- added joint y_thr_left: type None, limit lower=-7 upper=10
- added joint y_thr_right: type None, limit lower=-7 upper=10
- joint x_thr_left: limit lower=-30 upper=30 -> lower=-7 upper=10
- joint x_thr_right: limit lower=-30.0 upper=30.0 -> lower=-7 upper=10

Commit message: enabled Lidar (visual) and added two ballasts to balance Mallard

File: urdf/mallard_main.xacro (robot description, xacro)
@@ -126,5 +126,5 @@
     <child link="base_link"/>
   </joint> -->
-  <!-- <link name="lidar">
+  <link name="lidar">
     <visual name="lidar_base">
       <geometry>
@@ -154,13 +154,52 @@
     </collision>
     <inertial>
-      <mass value="0.250"/>
+      <mass value="0.25"/>
       <inertia ixx="0.00020" ixy="0.0" ixz="0.0" iyy="0.00020" iyz="0.0" izz="0.00015"/>
     </inertial>
-  </link> -->
-  <!-- <joint name="lidar_to_base_link" type="fixed">
+  </link>
+  <joint name="lidar_to_base_link" type="fixed">
     <parent link="base_link"/>
     <child link="lidar"/>
     <origin xyz="0.225 0.0 0.152" rpy="0.0 0.0 0.0"/>
-  </joint> -->
+  </joint>
+  <link name="ballast_1">
+    <visual name="">
+      <geometry>
+        <sphere radius="0.01"/>
+      </geometry>
+      <material name="red">
+        <color rgba="0.8 0.0 0.0 1.0"/>
+      </material>
+    </visual>
+    <inertial>
+      <mass value="0.11"/>
+      <inertia ixx="0" ixy="0" ixz="0" iyy="0" iyz="0" izz="0"/>
+    </inertial>
+  </link>
+  <link name="ballast_2">
+    <visual name="">
+      <geometry>
+        <sphere radius="0.01"/>
+      </geometry>
+      <material name="red">
+        <color rgba="0.8 0.0 0.0 1.0"/>
+      </material>
+    </visual>
+    <inertial>
+      <mass value="0.02"/>
+      <inertia ixx="0" ixy="0" ixz="0" iyy="0" iyz="0" izz="0"/>
+    </inertial>
+  </link>
+<!-- <origin xyz="0.225 0 0.076"> -->
+  <joint name="ballast_1_to_base_link" type="fixed">
+    <origin xyz="0.225 -0.25 0.076"/>
+    <parent link="base_link"/>
+    <child link="ballast_1"/>
+  </joint>
+   <joint name="ballast_2_to_base_link" type="fixed">
+    <origin xyz="-0.225 -0.25 0.076"/>
+    <parent link="base_link"/>
+    <child link="ballast_2"/>
+  </joint>
   <!-- Forward thrusters -->
   <xacro:thruster_link name="x_thr_left"   xyz="${(tl1/2)-0.188}  0.207 -0.041" rpy="0 ${-PI/2} 0"/>

Commit message: moved ballast and thruster links and joints to separate files. Cleaned up a little

File: urdf/mallard_main.xacro (robot description, xacro)
@@ -1,4 +1,6 @@
 <?xml version="1.0"?>
 <robot name="mallard" xmlns:xacro="http://www.ros.org/wiki/xacro">
+  <xacro:include filename="ballast.xacro"/>
+  <xacro:include filename="thruster.xacro"/>
   <!-- Thrusters components & constants -->
   <xacro:property name="PI" value="3.1415926535897931"/>
@@ -7,5 +9,5 @@
   <xacro:property name="tr2" value=".047" />
   <xacro:property name="tl2" value=".045" />
-  <material name="blue">
+  <!-- <material name="blue">
     <color rgba="0.0 0.0 0.8 1.0"/>
   </material>
@@ -18,8 +20,8 @@
   <material name="gray">
     <color rgba="0.8 0.8 0.8 1.0"/>
-  </material>
+  </material> -->
   <!--  *** MACROS *** -->
   <!-- Thruster link -->
-  <xacro:macro name="thruster_link" params="name xyz rpy">
+  <!-- <xacro:macro name="thruster_link" params="name xyz rpy">
       <joint name="${name}" type="revolute">
           <parent link="base_link"/>
@@ -31,5 +33,4 @@
       </joint>
       <link name="${name}">
-          <!-- <buoyancy><compensation>1.0</compensation></buoyancy> -->
           <visual name="${name}_1">
               <geometry>
@@ -41,5 +42,4 @@
           </visual>
           <visual name="${name}_2">
-              <!-- <origin xyz="0 0 ${(tl1+tl2)/2}"/> -->
               <origin xyz="0 0 ${tl2/4}"/>
               <geometry>
@@ -66,5 +66,5 @@
           <compensation>0.6</compensation>
       </buoyancy>
-  </xacro:macro>
+  </xacro:macro>  -->
   <!-- <link name="odom">
   </link> -->
@@ -75,9 +75,11 @@
           <box size="0.450 0.038 0.038"/>
         </geometry>
-        <material name="gray"/>
-        <origin  xyz="0 -0.15 0" rpy="0 0 0"/>
+        <material name="gray">
+          <color rgba="0.8 0.8 0.8 1.0"/>
+        </material>
+        <origin  xyz="0 -0.15 0" />
       </visual>
       <collision name="mallard_box">
-        <origin xyz="0 0 0.057" rpy="0 0 0"/>
+        <origin xyz="0 0 0.057"/>
         <geometry>
           <box size="0.564 0.5 0.152"/>
@@ -89,5 +91,5 @@
           <box size="0.450 0.038 0.038"/>
         </geometry>
-        <origin xyz="0 0.15 0" rpy="0 0 0"/>
+        <origin xyz="0 0.15 0" />
       </visual>
       <!-- Cylinders (acrylic tubes)-->
@@ -96,5 +98,5 @@
           <cylinder radius="0.057" length="0.5"/>
         </geometry>
-        <origin xyz="0.225 0 0.076" rpy="1.5707 0.0 0.0"/>
+        <origin xyz="0.225 0 0.076" rpy="1.5707 0 0"/>
       </visual>
       <visual name="rear_tube_visual">
@@ -102,5 +104,5 @@
           <cylinder radius="0.057" length="0.5"/>
         </geometry>
-        <origin xyz="-0.225 0 0.076" rpy="1.5707 0.0 0.0"/>
+        <origin xyz="-0.225 0 0.076" rpy="1.5707 0 0"/>
       </visual>
       <!-- chassis physics -->
@@ -117,6 +119,6 @@
           <compensation>1.2</compensation>
           <origin xyz= "0 0 0"/>
-          <limit radius="0.0"/>
-          <damping xyz="50 50 80" rpy="1 1 1"/>
+          <limit radius="0.1"/>
+          <damping xyz="100 100 100" rpy="2 2 2"/>
       </buoyancy>
   </link>
@@ -131,5 +133,7 @@
         <box size="0.06 0.061 0.048"/>
       </geometry>
-      <material name="blue"/>
+      <material name="blue">
+        <color rgba="0.0 0.0 0.8 1.0"/>
+      </material>
       <origin xyz="0.0 0.0 0.0"/>
     </visual>
@@ -141,18 +145,20 @@
     </collision>
     <visual name="optical_hood">
+      <origin xyz="0 0 0.0425"/>
       <geometry>
         <cylinder radius="0.025" length="0.037"/>
       </geometry>
-      <material name="blue"/>
-      <origin xyz="0.0 0.0 0.048"/>
+      <material name="blue">
+        <color rgba="0.0 0.0 0.8 1.0"/>
+      </material>
     </visual>
     <collision>
+      <origin xyz="0.0 0.0 0.048"/>
       <geometry>
         <cylinder radius="0.025" length="0.037"/>
       </geometry>
-      <origin xyz="0.0 0.0 0.048"/>
     </collision>
     <inertial>
-      <mass value="0.25"/>
+      <mass value="0.3"/>
       <inertia ixx="0.00020" ixy="0.0" ixz="0.0" iyy="0.00020" iyz="0.0" izz="0.00015"/>
     </inertial>
@@ -161,45 +167,9 @@
     <parent link="base_link"/>
     <child link="lidar"/>
-    <origin xyz="0.225 0.0 0.152" rpy="0.0 0.0 0.0"/>
+    <origin xyz="0.225 0 0.152"/>
   </joint>
-  <link name="ballast_1">
-    <visual name="">
-      <geometry>
-        <sphere radius="0.01"/>
-      </geometry>
-      <material name="red">
-        <color rgba="0.8 0.0 0.0 1.0"/>
-      </material>
-    </visual>
-    <inertial>
-      <mass value="0.11"/>
-      <inertia ixx="0" ixy="0" ixz="0" iyy="0" iyz="0" izz="0"/>
-    </inertial>
-  </link>
-  <link name="ballast_2">
-    <visual name="">
-      <geometry>
-        <sphere radius="0.01"/>
-      </geometry>
-      <material name="red">
-        <color rgba="0.8 0.0 0.0 1.0"/>
-      </material>
-    </visual>
-    <inertial>
-      <mass value="0.02"/>
-      <inertia ixx="0" ixy="0" ixz="0" iyy="0" iyz="0" izz="0"/>
-    </inertial>
-  </link>
-<!-- <origin xyz="0.225 0 0.076"> -->
-  <joint name="ballast_1_to_base_link" type="fixed">
-    <origin xyz="0.225 -0.25 0.076"/>
-    <parent link="base_link"/>
-    <child link="ballast_1"/>
-  </joint>
-   <joint name="ballast_2_to_base_link" type="fixed">
-    <origin xyz="-0.225 -0.25 0.076"/>
-    <parent link="base_link"/>
-    <child link="ballast_2"/>
-  </joint>
+  <!-- Ballast -->
+  <xacro:ballast name="ballast_1" mass="0.14" xyz=" 0.225 -0.25 0.076" rpy="${PI/2} 0 0"/>
+  <xacro:ballast name="ballast_2" mass="0.02" xyz="-0.225 -0.25 0.076" rpy="${PI/2} 0 0"/>
   <!-- Forward thrusters -->
   <xacro:thruster_link name="x_thr_left"   xyz="${(tl1/2)-0.188}  0.207 -0.041" rpy="0 ${-PI/2} 0"/>

Commit message: cleaned up main.xacro, removed dummy odom link and lidar body

File: urdf/mallard_main.xacro (robot description, xacro)
@@ -15,9 +15,4 @@
       <material>Gazebo/Blue</material>
   </gazebo>
-  <!-- <link name="odom">
-    <geometry>
-      <box size="0.01 0.01 0.01"/>
-    </geometry>
-  </link> -->
   <link name="base_link">
       <!-- Channels (aluminum connecting elements) -->
@@ -73,10 +68,4 @@
       </buoyancy>
   </link>
-  <!-- <joint name="odom_to_base_link" type="fixed">
-    <origin xyz="0.0 0.0 0.0" rpy="0.0 0.0 0.0"/>
-    <parent link="odom"/>
-    <child link="base_link"/>
-  </joint> -->
-  <!-- <xacro:lidar_body name="lidar_base" mass="0.27" xyz="0.225 0 0.152"/> -->
   <xacro:lidar
 		parent="base_link"

Commit message: small modifications to goal selector

File: urdf/mallard_main.xacro (robot description, xacro)
@@ -52,5 +52,5 @@
       <inertial>
         <origin xyz="0 0 -0.019" rpy="0 0 0"/>
-        <mass value="10.5"/>
+        <mass value="15.5"/>
         <inertia ixx="0.17" ixy="0.0" ixz="0.0" iyy="0.25" iyz="0.0" izz="0.40"/>
       </inertial>
@@ -59,5 +59,5 @@
       <buoyancy>
           <!-- Compensation coefficient is buoyancy force to weight ratio. Mallard
-               buoyancy force is 11.52kg, weight is10.5kg.   -->
+               buoyancy force is 12.6kg, weight is10.5kg.   -->
           <compensation>1.2</compensation>
           <origin xyz= "0 0 0"/>

Commit message: deleted old launch and .pyc files

File: urdf/mallard_main.xacro (robot description, xacro)
@@ -52,5 +52,5 @@
       <inertial>
         <origin xyz="0 0 -0.019" rpy="0 0 0"/>
-        <mass value="15.5"/>
+        <mass value="10.5"/>
         <inertia ixx="0.17" ixy="0.0" ixz="0.0" iyy="0.25" iyz="0.0" izz="0.40"/>
       </inertial>

Commit message: finished testing step PYTHON script that launches,records rosbags and changes URDF file. Again it is for open-loop step response

File: urdf/mallard_main.xacro (robot description, xacro)
@@ -52,5 +52,5 @@
       <inertial>
         <origin xyz="0 0 -0.019" rpy="0 0 0"/>
-        <mass value="10.5"/>
+        <mass value="8.0"/>
         <inertia ixx="0.17" ixy="0.0" ixz="0.0" iyy="0.25" iyz="0.0" izz="0.40"/>
       </inertial>
