Commit message: got to publish and subscribe to controllers in gazebo via ROS. Whats left is to specify physics so actuator has friction and moves mallard

File: urdf/archive/01-chassis.urdf (robot description, URDF)
Before this commit: robot mallard_origins, 3 links, 2 joints
Links:
- link lidar: mass None -> 0.250; geometry collision box size=0.06 0.061 0.048; collision cylinder length=0.037 radius=0.025
