Commit message: finished urdf file mass update cycle

File: py_launch/mallard_main.xacro (robot description, xacro)
@@ -52,5 +52,5 @@
       <inertial>
         <origin xyz="0 0 -0.019" rpy="0 0 0"/>
-        <mass value="14.0"/>
+        <mass value="10.5"/>
         <inertia ixx="0.17" ixy="0.0" ixz="0.0" iyy="0.25" iyz="0.0" izz="0.40"/>
       </inertial>
